File: display.kicad_sch (KiCad schematic)
At the start: 10 parts, among them Q1 ZXM61N03F, U1 E2206KS0E1

Commit message: 2nd display
Parts:
- added U2: E2206KS0E1, symbol rsx_misc:Graphic Display
Changed lines of the file:
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@@
+	)
+	(symbol
+		(lib_name "Graphic Display_1")
+		(lib_id "rsx_misc:Graphic Display")
+		(at 67.31 76.2 0)
+		(unit 1)
+		(exclude_from_sim no)
+		(in_bom yes)
+		(on_board yes)
+		(dnp no)
+		(fields_autoplaced yes)
+		(property "Reference" "U2"
+			(at 101.6 106.0449 0)
+			(effects
+				(font
+					(size 1.524 1.524)
+				)
+				(justify left)
+			)
+		)
+		(property "Value" "E2206KS0E1"
+			(at 101.6 108.5849 0)
+			(effects
+				(font
+					(size 1.524 1.524)
+				)
+				(justify left)
+			)
+		)
+		(property "Footprint" ""
+			(at 67.31 76.2 0)
+			(effects
+				(font
+					(size 1.27 1.27)
+					(italic yes)
+				)
+				(hide yes)
+			)
+		)
+		(property "Datasheet" ""
+			(at 67.31 76.2 0)
+			(effects
+				(font
+					(size 1.27 1.27)
+					(italic yes)
+				)
+				(hide yes)
+			)
+		)
+		(property "Description" "GRAPHIC DISPLAY TFT BLACK 2.06\""
+			(at 67.31 76.2 0)
+			(effects
+				(font
+					(size 1.27 1.27)
+				)
+				(hide yes)
+			)
+		)
+		(property "dpn" "553-3758-ND"
+			(at 67.31 76.2 0)
+			(effects
+				(font
+					(size 1.27 1.27)
+				)
+				(hide yes)
+			)
+		)
+		(property "Manufacturer" "Pervasive Displays"
+			(at 67.31 76.2 0)
+			(effects
+				(font
+					(size 1.27 1.27)
+				)
+				(hide yes)
+			)
+		)
+		(property "Manufacture Product Number" "E2206KS0E1"
+			(at 67.31 76.2 0)
+			(effects
+				(font
+					(size 1.27 1.27)
+				)
+				(hide yes)
+			)
+		)
+		(pin "17"
+		)
+		(pin "22"
+		)
+		(pin "5"
+		)
+		(pin "7"
+		)
+		(pin "9"
+		)
+		(pin "1"
+		)
+		(pin "10"
+		)
+		(pin "18"
+		)
+		(pin "21"
+		)
+		(pin "4"
+		)
+		(pin "8"
+		)
+		(pin "3"
+		)
+		(pin "15"
+		)
+		(pin "6"
+		)
+		(pin "11"
+		)
+		(pin "2"
+		)
+		(pin "13"
+		)
+		(pin "16"
+		)
+		(pin "12"
+		)
+		(pin "14"
+		)
+		(pin "19"
+		)
+		(pin "20"
+		)
+		(pin "24"
+		)
+		(pin "23"
+		)
+		(instances
+			(project ""
+				(path "/a03b232e-bbf4-4c47-a930-a77d53fe4ba2"
+					(reference "U2")
+					(unit 1)
+				)
+			)
+		)
 	)
 	(symbol

Commit message: Update display.kicad_sch
Connections:
- net at U1.2: now also Q1.1 (G)
- net at U1.5: no longer C1.2
Other:
- moved on the sheet: C1, Q1
Changed lines of the file:
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@@
+	(wire
+		(pts
+			(xy 228.6 67.31) (xy 228.6 72.39)
+		)
+		(stroke
+			(width 0)
+			(type default)
+		)
+	)
 	(wire
 		(pts
@@
 	(wire
 		(pts
-			(xy 233.68 69.85) (xy 233.68 67.31)
-		)
-		(stroke
-			(width 0)
-			(type default)
-		)
-	)
-	(wire
-		(pts
 			(xy 207.01 93.98) (xy 236.22 93.98)
 		)
@@
 	(wire
 		(pts
-			(xy 233.68 67.31) (xy 238.76 67.31)
+			(xy 228.6 72.39) (xy 229.87 72.39)
+		)
+		(stroke
+			(width 0)
+			(type default)
+		)
+	)
+	(wire
+		(pts
+			(xy 215.9 59.69) (xy 238.76 59.69)
 		)
 		(stroke
@@
 	(symbol
 		(lib_id "Transistor_FET:ZXM61N03F")
-		(at 213.36 59.69 0)
+		(at 210.82 59.69 0)
 		(mirror y)
 		(unit 1)
@@
 		(dnp no)
 		(property "Reference" "Q1"
-			(at 207.01 60.9601 0)
+			(at 204.47 60.9601 0)
 			(effects
 				(font
@@
 		)
 		(property "Value" "ZXM61N03F"
-			(at 207.01 58.4201 0)
+			(at 204.47 58.4201 0)
 			(effects
 				(font
@@
 		)
 		(property "Footprint" "Package_TO_SOT_SMD:SOT-23"
-			(at 208.28 61.595 0)
+			(at 205.74 61.595 0)
 			(effects
 				(font
@@
 		)
 		(property "Datasheet" "http://www.diodes.com/assets/Datasheets/ZXM61N03F.pdf"
-			(at 208.28 63.5 0)
+			(at 205.74 63.5 0)
 			(effects
 				(font
@@
 		)
 		(property "Description" "1.4A Id, 30V Vds, N-Channel MOSFET, SOT-23"
-			(at 213.36 59.69 0)
+			(at 210.82 59.69 0)
 			(effects
 				(font
@@
 	(symbol
 		(lib_id "rsx_Capacitors:1u")
-		(at 229.87 69.85 90)
+		(at 224.79 67.31 90)
 		(unit 1)
 		(exclude_from_sim no)
@@
 		(on_board yes)
 		(dnp no)
-		(fields_autoplaced yes)
 		(property "Reference" "C1"
-			(at 229.87 62.23 90)
+			(at 227.33 66.04 90)
 			(effects
 				(font
@@
 		)
 		(property "Value" "1u"
-			(at 229.87 64.77 90)
+			(at 227.33 68.58 90)
 			(effects
 				(font
@@
 		)
 		(property "Footprint" "rsx_capacitors:C_0805_2012Metric"
-			(at 233.68 68.8848 0)
+			(at 228.6 66.3448 0)
 			(effects
 				(font
@@
 		)
 		(property "Datasheet" "~"
-			(at 229.87 69.85 0)
+			(at 224.79 67.31 0)
 			(effects
 				(font
@@
 		)
 		(property "Description" "CAP CER 1UF 50V X7R 0805"
-			(at 229.87 69.85 0)
+			(at 224.79 67.31 0)
 			(effects
 				(font
@@
 		)
 		(property "MFR" "Samsung Electro-Mechanics"
-			(at 229.87 69.85 0)
+			(at 224.79 67.31 0)
 			(effects
 				(font
@@
 		)
 		(property "DPN" "1276-1029-1-ND"
-			(at 229.87 69.85 0)
+			(at 224.79 67.31 0)
 			(effects
 				(font
@@
 		)
 		(property "MPN" "CL21B105KBFNNNE"
-			(at 229.87 69.85 0)
-			(effects
-				(font
+			(at 224.79 67.31 0)
+			(effects
+				(font

Commit message: Update display.kicad_sch
Connections:
- net at R1.1: now also C1.1
- net at R1.2: now also Q1.2 (S), U1.3
- net at U1.5: now also C1.2
Other:
- moved on the sheet: Q1, R1
Changed lines of the file:
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@@
 	(paper "A4")
+	(junction
+		(at 208.28 62.23)
+		(diameter 0)
+		(color 0 0 0 0)
+	)
 	(junction
 		(at 186.69 111.76)
@@
 	(wire
 		(pts
-			(xy 228.6 67.31) (xy 228.6 72.39)
+			(xy 217.17 57.15) (xy 217.17 59.69)
 		)
 		(stroke
@@
 	(wire
 		(pts
+			(xy 217.17 59.69) (xy 238.76 59.69)
+		)
+		(stroke
+			(width 0)
+			(type default)
+		)
+	)
+	(wire
+		(pts
+			(xy 200.66 62.23) (xy 208.28 62.23)
+		)
+		(stroke
+			(width 0)
+			(type default)
+		)
+	)
+	(wire
+		(pts
 			(xy 238.76 96.52) (xy 236.22 96.52)
 		)
@@
 	(wire
 		(pts
+			(xy 220.98 67.31) (xy 190.5 67.31)
+		)
+		(stroke
+			(width 0)
+			(type default)
+		)
+	)
+	(wire
+		(pts
 			(xy 186.69 116.84) (xy 210.82 116.84)
 		)
@@
 	(wire
 		(pts
+			(xy 190.5 62.23) (xy 193.04 62.23)
+		)
+		(stroke
+			(width 0)
+			(type default)
+		)
+	)
+	(wire
+		(pts
 			(xy 236.22 96.52) (xy 236.22 93.98)
 		)
@@
 	(wire
 		(pts
+			(xy 228.6 67.31) (xy 238.76 67.31)
+		)
+		(stroke
+			(width 0)
+			(type default)
+		)
+	)
+	(wire
+		(pts
 			(xy 186.69 116.84) (xy 186.69 138.43)
 		)
@@
 	(wire
 		(pts
-			(xy 228.6 72.39) (xy 229.87 72.39)
-		)
-		(stroke
-			(width 0)
-			(type default)
-		)
-	)
-	(wire
-		(pts
-			(xy 215.9 59.69) (xy 238.76 59.69)
+			(xy 215.9 57.15) (xy 217.17 57.15)
+		)
+		(stroke
+			(width 0)
+			(type default)
+		)
+	)
+	(wire
+		(pts
+			(xy 190.5 67.31) (xy 190.5 62.23)
 		)
 		(stroke
@@
 		(pts
 			(xy 186.69 101.6) (xy 186.69 106.68)
+		)
+		(stroke
+			(width 0)
+			(type default)
+		)
+	)
+	(wire
+		(pts
+			(xy 208.28 62.23) (xy 238.76 62.23)
 		)
 		(stroke
@@
 	(symbol
 		(lib_id "rsx_Resistors:0.47R")
-		(at 196.85 80.01 90)
+		(at 196.85 62.23 90)
 		(unit 1)
 		(exclude_from_sim no)
@@
 		(fields_autoplaced yes)
 		(property "Reference" "R1"
-			(at 196.85 73.66 90)
+			(at 196.85 55.88 90)
 			(effects
 				(font
@@
 		)
 		(property "Value" "0.47R"
-			(at 196.85 76.2 90)
+			(at 196.85 58.42 90)
 			(effects
 				(font
@@
 		)
 		(property "Footprint" "rsx_resistors:R_1206_3216Metric"
-			(at 196.85 81.788 90)
+			(at 196.85 64.008 90)
 			(effects
 				(font
@@
 		)
 		(property "Datasheet" "https://www.yageogroup.com/content/Resource%20Library/Datasheet/PYU-RL_GROUP_521_ROHS_L.pdf"
-			(at 196.85 80.01 0)
+			(at 196.85 62.23 0)
 			(effects
 				(font
@@
 		)
 		(property "Description" "RES 0.47 OHM 1% 1/4W 1206"
-			(at 196.85 80.01 0)
+			(at 196.85 62.23 0)
 			(effects
 				(font
@@
 		)
 		(property "MFR" "  YAGEO"
-			(at 196.85 80.01 0)
+			(at 196.85 62.23 0)
 			(effects
 				(font
@@
 		)
 		(property "DPN" "311-.47LWCT-ND"
-			(at 196.85 80.01 0)
+			(at 196.85 62.23 0)
 			(effects
 				(font
@@
 		)
 		(property "MPN" "RL1206FR-070R47L"
-			(at 196.85 80.01 0)
+			(at 196.85 62.23 0)
 			(effects
 				(font
@@
 	(symbol
 		(lib_id "Transistor_FET:ZXM61N03F")
-		(at 210.82 59.69 0)
+		(at 210.82 57.15 0)
 		(mirror y)
 		(unit 1)
@@
 		(dnp no)
 		(property "Reference" "Q1"
-			(at 204.47 60.9601 0)
+			(at 214.884 52.578 0)
 			(effects
 				(font
@@
 		)
 		(property "Value" "ZXM61N03F"
-			(at 204.47 58.4201 0)
+			(at 214.884 50.038 0)
 			(effects
 				(font
@@
 		)
 		(property "Footprint" "Package_TO_SOT_SMD:SOT-23"
-			(at 205.74 61.595 0)
+			(at 205.74 59.055 0)
 			(effects
 				(font
@@
 		)
 		(property "Datasheet" "http://www.diodes.com/assets/Datasheets/ZXM61N03F.pdf"
-			(at 205.74 63.5 0)
+			(at 205.74 60.96 0)
 			(effects
 				(font
@@
 		)
 		(property "Description" "1.4A Id, 30V Vds, N-Channel MOSFET, SOT-23"
-			(at 210.82 59.69 0)
-			(effects
-				(font
+			(at 210.82 57.15 0)
+			(effects
+				(font
