File: battery_display/battery_display.kicad_sch (KiCad schematic)
At the start: 0 parts

Commit message: started battery display schematic
Parts:
- added J1: FH34SRJ-24S-0.5SH_99_, rsx_headers_communications:HRS_FH34SRJ-24S-0.5SH_99_, symbol rsx_Header_communication:FH34SRJ-24S-0.5SH_99_
- added Q1: ZXM61N03F, rsx_packages_TO_SOT:SOT-23, symbol rsx_Transistors:ZXM61N03F
- added R1: 0.47R, rsx_resistors:R_1206_3216Metric, symbol rsx_Resistors:0.47R
Connections:
- new net: J1.2, Q1.1 (G)
- new net: J1.3, Q1.2 (S), R1.2
- new net: J1.5, R1.1
- no-connect marks 0 -> 5
