File: battery_display/battery_display.kicad_pcb (KiCad board)
At the start: 2 copper layers, 100 x 60 mm, 30 parts, among them J1 FH34SRJ-24S-0.5SH_99_, J2 Screw_Terminal_2x2.54, Q1 ZXM61N03F, Q2 ZXM61N03F, SW1 Button-THT - 2-1825910-7, U1 LDO40LPU33RY

Commit message: actually made the changes in the previous 2 pushes
💀
Parts:
- moved H1 37.0 mm to (185.0, 38.0)
- moved H2 36.5 mm to (185.0, 83.0)
- moved U1 12.8 mm to (197.9, 37.1)
- moved J2 12.8 mm to (223.2, 34.5)
- moved R4 12.8 mm to (196.2, 32.5)
- moved C10 12.8 mm to (193.0, 40.0)
- moved C12 12.8 mm to (201.3, 37.0)
- moved C13 12.8 mm to (193.8, 37.0)
- moved C9 12.8 mm to (193.8, 41.5)
- moved R3 12.8 mm to (200.0, 32.5)
- moved SW1 12.8 mm to (214.8, 37.3)
Routing:
- net /read_voltage: track 97.5 -> 31.5 mm
- net /Display VDDD: track 55.7 -> 69.3 mm
- net /BS: track 76.3 -> 78.7 mm, vias 1 -> 2
- net /panelDC: vias 1 -> 2
- net /panelBusy: vias 1 -> 2
- net /panelReset: vias 1 -> 2
- net /panelCS: vias 1 -> 2
- net /SDA: vias 1 -> 2
- net /SCLK: vias 1 -> 2
