File: witharduinoandnewcomps/_autosave-witharduinoandnewcomps.kicad_sch (KiCad schematic)
At the start: 27 parts, among them J1 FH34SRJ-24S-0.5SH_99_, Q1 ZXM61N03F, Q3 ZXM61N03F, SW1 Button-THT - 2-1825910-7, U1 LDO40LPU33RY

Commit message: Nov22
Parts:
- added J2: Screw_Terminal_2x2.54, rsx_headers_screw:Wurth_691210910002, symbol rsx_header_screw:Screw_Terminal_2x2.54
Connections:
- net +12V: no longer SW1.1
- net GND: now also A1.13 (GND), A1.18 (GND), A1.23 (GND), A1.28 (GND), A1.3 (GND), A1.38 (GND), A1.8 (GND)
- net GNDPWR: now also J2.2 (Pin_2); no longer A1.13 (GND), A1.18 (GND), A1.23 (GND), A1.28 (GND), A1.3 (GND), A1.38 (GND), A1.8 (GND)
- new net: J2.1 (Pin_1), SW1.1
- no-connect marks 7 -> 33
