File: witharduinoandnewcomps/witharduinoandnewcomps.kicad_sch (KiCad schematic)
At the start: 27 parts, among them J1 FH34SRJ-24S-0.5SH_99_, Q1 ZXM61N03F, Q3 ZXM61N03F, SW1 Button-THT - 2-1825910-7, U1 LDO40LPU33RY

Commit message: laid out pcb
Parts:
- removed C10: 4u7, rsx_capacitors:C_0805_2012Metric, symbol rsx_Capacitors:4u7
- added C14: 4u7, rsx_capacitors:C_0805_2012Metric, symbol rsx_Capacitors:4u7
- added J3: Screw_Terminal_2x2.54, rsx_headers_screw:Wurth_691210910002, symbol rsx_header_screw:Screw_Terminal_2x2.54
Connections:
- net GNDPWR is gone; now on net GND: A1.13 (GND), A1.18 (GND), A1.23 (GND), A1.28 (GND), A1.3 (GND), A1.38 (GND), A1.8 (GND), C1.1, C2.1, C3.1, C4.1, C5.1, C6.1, C7.1, C8.1, C9.2, CR2.1, J1.17, R1.1, R3.2
- net +12V: now also J3.1 (Pin_1)
- net 3.3v in power: now also C13.1, U1.5 (Vsense)
- net GND: now also J1.S1 (SHIELD), J1.S2 (SHIELD__1), J3.2 (Pin_2)
- net at CR1.2, Q3.3 (D), SRP3012TA-100M1.2: now also C14.1
- net at R3.1, R4.2: now also A1.31 (GPIO26_ADC0); no longer A1.34 (GPIO28_ADC2)
- net at CR2.2, CR4.1: now also C14.2
- new net: C6.2, CR4.2, J1.23
- new net: C2.2, J1.24
- no-connect marks 7 -> 31
Other:
- note added: "display connector"
- note added: "read voltage"
- note added: "soft start"
- note added: "voltage divider"
- note added: "voltage regulator"
- moved on the sheet: C12
