File: FinalBatteryDisplay/ConnectedRedoJan24BatteryDisplaySchem.kicad_pcb (KiCad board)
At the start: 2 copper layers, 97 x 60 mm, 27 parts, among them J1 FH34SRJ-24S-0.5SH_99_, J2 Screw_Terminal_2x2.54, Q2 ZXM61N03F, SW1 Button

Commit message: Drill, Gerber and BOM
Routing:
- net Net-(Q2-D): track 3.50 -> 24.1 mm, vias 0 -> 2
- net GND: track 66.2 -> 81.5 mm, vias 4 -> 5
- net SDA: track 45.6 -> 40.7 mm, vias 1 -> 2
- net CSB: track 33.1 -> 28.9 mm
- net SCL: track 38.3 -> 36.0 mm
- net Net-(Q2-G): track 27.6 -> 25.5 mm
- net Net-(C1-Pad2): track 22.1 -> 22.7 mm

Commit message: layout update
Parts:
- moved C13 2.89 mm to (158.5, 50.0)
- moved C7 1.69 mm to (159.5, 47.0), turned to 0 degrees
Routing:
- net GND: track 81.5 -> 78.5 mm
- net +3.3V: track 116.6 -> 116.0 mm
Other:
- board text added: "12V"
- board text added: "GND"
- board text added: "Helen (2026)"
