File: NewNewDisplay/RevisedYey/_autosave-RevisedYey.kicad_sch (KiCad schematic)
At the start: 29 parts, among them J1 Screw_Terminal_2x2.54, J3 FH34SRJ-24S-0.5SH_99_, Q1 ZXM61N03F, SW2 Button-THT - 2-1825910-7

Commit message: PCB_Done
Connections:
- no-connect marks 32 -> 31
Changed lines of the file:
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@@
-	)
-	(no_connect
-		(at 101.6 124.46)
 	)
 	(no_connect
